File: Polygonus-Universal-Base.kicad_pcb (KiCad board)
At the start: 2 copper layers, 160 x 118 mm, 51 parts, among them J4 Polygonus_Plugs, J5 Conn_02x04_Top_Bottom, Q1 NGD8201AN, Q2 NGD8201AN, Q3 NGD8201AN, Q4 NGD8201AN, Q5 NGD8201AN, Q6 NGD8201AN, Q7 NGD8201AN, Q8 NGD8201AN, U1 WBO-Single-Module, U10 VNL5090, U11 VNL5090, U12 VNL5090, U2 TLE9201SG, U3 MAX9924, U4 VNL5090, U5 VNL5090, U6 VNL5090, U7 VNL5090, U8 TLE9201SG, U9 VNL5090

Commit message: Made the board
Parts:
- removed JP1: Jumper_2_Open, Resistor_THT:R_Axial_DIN0309_L9.0mm_D3.2mm_P15.24mm_Horizontal
- J4: footprint Simon:Polygonus_Plugs -> Simon:Polygonus-With-USB-SWD
- moved U10 179.8 mm to (68.3, 62.1), turned to 0 degrees
- moved U11 172.4 mm to (68.3, 77.6), turned to 0 degrees
- moved RN3 169.4 mm to (60.2, 72.3)
- moved U12 168.5 mm to (68.3, 69.7), turned to 0 degrees
- moved U9 164.3 mm to (68.3, 54.7), turned to 0 degrees
- moved RN4 161.7 mm to (74.6, 73.3)
- moved C9 117.0 mm to (108.4, 42.2)
- moved U8 104.8 mm to (115.7, 45.4), turned to 180 degrees
- moved C8 100.8 mm to (124.1, 42.8), turned to 180 degrees
- moved C3 96.5 mm to (91.6, 44.1), turned to -90 degrees
- moved R12 94.0 mm to (122.2, 50.6), turned to 90 degrees
- moved C7 93.7 mm to (125.2, 46.5), turned to 90 degrees
- moved C2 90.8 mm to (106.7, 43.2), turned to 90 degrees
- moved U2 88.4 mm to (98.9, 45.6), turned to 180 degrees
- moved C1 82.8 mm to (106.6, 47.6), turned to 90 degrees
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Connections:
- C1 pad 2: /12V_MR_FUSE -> /12V_MR
- C7 pad 2: /12V_MR_FUSE -> /12V_MR
- J5 pad 1: /LSU_12v -> /12V_MR_FUSE
- J5 pad 2: /LSU_12v -> /12V_MR_FUSE
- Motronic_88pin1 pad 1: unconnected-(Motronic_88pin1-Pad1) -> /ExtraLSA
- Motronic_88pin1 pad 10: unconnected-(Motronic_88pin1-Pad10) -> /12V_MR
- Motronic_88pin1 pad 11: unconnected-(Motronic_88pin1-Pad11) -> /AV2
- Motronic_88pin1 pad 12: unconnected-(Motronic_88pin1-Pad12) -> /AV5
- Motronic_88pin1 pad 13: unconnected-(Motronic_88pin1-Pad13) -> /AV8
- Motronic_88pin1 pad 14: unconnected-(Motronic_88pin1-Pad14) -> /AV11
- Motronic_88pin1 pad 15: unconnected-(Motronic_88pin1-Pad15) -> /AT1
- Motronic_88pin1 pad 16: unconnected-(Motronic_88pin1-Pad16) -> /AT4
- Motronic_88pin1 pad 2: unconnected-(Motronic_88pin1-Pad2) -> /ExtraLSC
- Motronic_88pin1 pad 21: unconnected-(Motronic_88pin1-Pad21) -> /12V_KEY
- Motronic_88pin1 pad 22: unconnected-(Motronic_88pin1-Pad22) -> /IGBT7
- Motronic_88pin1 pad 23: unconnected-(Motronic_88pin1-Pad23) -> /IGBT5
- Motronic_88pin1 pad 24: unconnected-(Motronic_88pin1-Pad24) -> /IGBT3
- Motronic_88pin1 pad 25: unconnected-(Motronic_88pin1-Pad25) -> /IGBT1
- Motronic_88pin1 pad 26: unconnected-(Motronic_88pin1-Pad26) -> /LS10ADD
- Motronic_88pin1 pad 27: unconnected-(Motronic_88pin1-Pad27) -> /LS12ADD
- Motronic_88pin1 pad 28: unconnected-(Motronic_88pin1-Pad28) -> /12V_MR
- Motronic_88pin1 pad 29: unconnected-(Motronic_88pin1-Pad29) -> /ExtraLSB
- Motronic_88pin1 pad 3: unconnected-(Motronic_88pin1-Pad3) -> /HS4
- Motronic_88pin1 pad 30: unconnected-(Motronic_88pin1-Pad30) -> /ExtraLSD
- Motronic_88pin1 pad 31: unconnected-(Motronic_88pin1-Pad31) -> /HS3
- Motronic_88pin1 pad 32: unconnected-(Motronic_88pin1-Pad32) -> /HS1
- Motronic_88pin1 pad 33: unconnected-(Motronic_88pin1-Pad33) -> /ETB2_+
- Motronic_88pin1 pad 34: unconnected-(Motronic_88pin1-Pad34) -> /ETB1_+
- Motronic_88pin1 pad 35: unconnected-(Motronic_88pin1-Pad35) -> /KNOCK_1
- Motronic_88pin1 pad 37: unconnected-(Motronic_88pin1-Pad37) -> /12V_MR
- Motronic_88pin1 pad 38: unconnected-(Motronic_88pin1-Pad38) -> /AV1
- Motronic_88pin1 pad 39: unconnected-(Motronic_88pin1-Pad39) -> /AV4
- Motronic_88pin1 pad 4: unconnected-(Motronic_88pin1-Pad4) -> /HS2
- Motronic_88pin1 pad 40: unconnected-(Motronic_88pin1-Pad40) -> /AV7
- Motronic_88pin1 pad 41: unconnected-(Motronic_88pin1-Pad41) -> /CRANK +
- Motronic_88pin1 pad 42: unconnected-(Motronic_88pin1-Pad42) -> /CRANK -
- Motronic_88pin1 pad 43: unconnected-(Motronic_88pin1-Pad43) -> /AT3
- Motronic_88pin1 pad 49: unconnected-(Motronic_88pin1-Pad49) -> /IGBT8
- Motronic_88pin1 pad 5: unconnected-(Motronic_88pin1-Pad5) -> /ETB2_-
- Motronic_88pin1 pad 50: unconnected-(Motronic_88pin1-Pad50) -> /IGBT6
- Motronic_88pin1 pad 51: unconnected-(Motronic_88pin1-Pad51) -> /IGBT4
- Motronic_88pin1 pad 52: unconnected-(Motronic_88pin1-Pad52) -> /IGBT2
- Motronic_88pin1 pad 53: unconnected-(Motronic_88pin1-Pad53) -> /LS9ADD
- Motronic_88pin1 pad 54: unconnected-(Motronic_88pin1-Pad54) -> /LS11ADD
- Motronic_88pin1 pad 55: unconnected-(Motronic_88pin1-Pad55) -> GND
- Motronic_88pin1 pad 56: unconnected-(Motronic_88pin1-Pad56) -> /5V_SENSOR_2
- Motronic_88pin1 pad 57: unconnected-(Motronic_88pin1-Pad57) -> /5V_SENSOR_2
- Motronic_88pin1 pad 58: unconnected-(Motronic_88pin1-Pad58) -> /5V_SENSOR_1
- Motronic_88pin1 pad 59: unconnected-(Motronic_88pin1-Pad59) -> /5V_SENSOR_1
- Motronic_88pin1 pad 6: unconnected-(Motronic_88pin1-Pad6) -> /ETB1_-
- Motronic_88pin1 pad 60: unconnected-(Motronic_88pin1-Pad60) -> /DIGITAL_6
- Motronic_88pin1 pad 61: unconnected-(Motronic_88pin1-Pad61) -> /DIGITAL_5
- Motronic_88pin1 pad 62: unconnected-(Motronic_88pin1-Pad62) -> /DIGITAL_4
- Motronic_88pin1 pad 63: unconnected-(Motronic_88pin1-Pad63) -> /DIGITAL_3
- Motronic_88pin1 pad 64: unconnected-(Motronic_88pin1-Pad64) -> /DIGITAL_2
- Motronic_88pin1 pad 65: unconnected-(Motronic_88pin1-Pad65) -> /DIGITAL_1
- Motronic_88pin1 pad 68: unconnected-(Motronic_88pin1-Pad68) -> /12V_MR
- Motronic_88pin1 pad 69: unconnected-(Motronic_88pin1-Pad69) -> /AV3
- Motronic_88pin1 pad 7: unconnected-(Motronic_88pin1-Pad7) -> /KNOCK_2
- Motronic_88pin1 pad 70: unconnected-(Motronic_88pin1-Pad70) -> /AV6
- Motronic_88pin1 pad 71: unconnected-(Motronic_88pin1-Pad71) -> /AV9
- Motronic_88pin1 pad 72: unconnected-(Motronic_88pin1-Pad72) -> /AV10
- Motronic_88pin1 pad 73: unconnected-(Motronic_88pin1-Pad73) -> /AT2
- Motronic_88pin1 pad 74: unconnected-(Motronic_88pin1-Pad74) -> /CAN-
- Motronic_88pin1 pad 75: unconnected-(Motronic_88pin1-Pad75) -> /CAN+
- Motronic_88pin1 pad 76: unconnected-(Motronic_88pin1-Pad76) -> /LS1
- Motronic_88pin1 pad 77: unconnected-(Motronic_88pin1-Pad77) -> /LS2
- Motronic_88pin1 pad 78: unconnected-(Motronic_88pin1-Pad78) -> /LS3
- Motronic_88pin1 pad 79: unconnected-(Motronic_88pin1-Pad79) -> /LS4
- Motronic_88pin1 pad 80: unconnected-(Motronic_88pin1-Pad80) -> /LS5
- Motronic_88pin1 pad 81: unconnected-(Motronic_88pin1-Pad81) -> /LS6
- Motronic_88pin1 pad 82: unconnected-(Motronic_88pin1-Pad82) -> /LS7
- Motronic_88pin1 pad 83: unconnected-(Motronic_88pin1-Pad83) -> /LS8
- Motronic_88pin1 pad 84: unconnected-(Motronic_88pin1-Pad84) -> /Perm_Live
- Motronic_88pin1 pad 85: unconnected-(Motronic_88pin1-Pad85) -> /LS16
- Motronic_88pin1 pad 86: unconnected-(Motronic_88pin1-Pad86) -> /LS15
- Motronic_88pin1 pad 87: unconnected-(Motronic_88pin1-Pad87) -> /LS14
- Motronic_88pin1 pad 88: unconnected-(Motronic_88pin1-Pad88) -> /LS13
- U2 pad 4: /12V_MR_FUSE -> /12V_MR
- U8 pad 4: /12V_MR_FUSE -> /12V_MR
Routing:
- net /IGN10: track 0.00 -> 228.0 mm, vias 0 -> 3
- net /IGN9: track 0.00 -> 226.2 mm, vias 0 -> 3
- net /IGN11: track 0.00 -> 226.2 mm, vias 0 -> 3
- net /IGN12: track 0.00 -> 223.0 mm, vias 0 -> 3
- net /HS4: track 0.00 -> 206.4 mm
- net /HS3: track 0.00 -> 201.3 mm
- net /HS2: track 0.00 -> 198.5 mm
- net /HS1: track 0.00 -> 194.8 mm
- net /5V_SENSOR_2: track 86.0 -> 280.6 mm
- net /5V_SENSOR_1: track 0.00 -> 180.9 mm
- net /Perm_Live: track 0.00 -> 172.5 mm, vias 0 -> 2
- net /12V_MR: track 18.6 -> 157.3 mm, vias 0 -> 3
- net /12V_KEY: track 0.00 -> 132.8 mm
- net /+3V3: track 0.00 -> 123.1 mm, vias 0 -> 2
- net /VR1+: track 0.00 -> 121.8 mm, vias 0 -> 1
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
Commit message: Competed board
Parts:
- moved C9 0.24 mm to (108.4, 42.4)
- moved C2 0.16 mm to (106.8, 43.3)
Routing:
- net GND: track 0.00 -> 14.2 mm, vias 51 -> 496
- net /IGBT3: track 18.5 -> 21.1 mm
- net /VR1+: track 121.8 -> 124.3 mm
- net /IGN9: track 226.2 -> 228.7 mm
- net /12V_MR: track 157.3 -> 155.4 mm
- net /IGN10: track 228.0 -> 229.5 mm
- net /IGBT6: track 36.2 -> 37.6 mm
- net /IGBT4: track 33.9 -> 35.2 mm
- net /LS4: track 94.2 -> 95.4 mm
- net /IGBT7: track 22.5 -> 23.3 mm
- net /LS3: track 105.1 -> 105.9 mm
- net /IGBT8: track 39.8 -> 40.5 mm
- net /DIGITAL_1: track 80.0 -> 80.6 mm
- net /KNOCK_2: track 42.3 -> 42.9 mm
- net /ETB2_+: track 13.6 -> 14.2 mm

Commit message: upgraded
Parts:
- added C10: 1u, Resistor_SMD:R_0805_2012Metric, F.Cu at (135.2, 134.7)
- added C11: 56u, Capacitor_THT:CP_Radial_D8.0mm_P3.50mm, F.Cu at (101.1, 65.1)
- added C12: 47p, Capacitor_SMD:C_0805_2012Metric, F.Cu at (171.8, 143.0)
- added C13: 47p, Capacitor_SMD:C_0805_2012Metric, F.Cu at (174.1, 137.0)
- added C14: 100n, Capacitor_SMD:C_0805_2012Metric, F.Cu at (186.1, 142.4)
- added C15: 100n, Capacitor_SMD:C_0805_2012Metric, F.Cu at (178.8, 136.3)
- added C16: 47p, Capacitor_SMD:C_0805_2012Metric, F.Cu at (81.8, 137.6)
- added C17: 47p, Capacitor_SMD:C_0805_2012Metric, F.Cu at (81.2, 143.1)
- added C18: 100n, Capacitor_SMD:C_0805_2012Metric, F.Cu at (70.0, 139.1)
- added C19: 100n, Capacitor_SMD:C_0805_2012Metric, F.Cu at (68.3, 142.8)
- added D1: NUP2105L, Package_TO_SOT_SMD:SOT-23, F.Cu at (171.5, 140.1)
- added D2: NUP2105L, Package_TO_SOT_SMD:SOT-23, F.Cu at (86.0, 142.5)
- added J1: Conn_02x04_Top_Bottom, Connector_Molex:Molex_Micro-Fit_3.0_43045-0800_2x04_P3.00mm_Horizontal, F.Cu at (62.4, 103.1)
- added R13: DNP, Resistor_SMD:R_0805_2012Metric, F.Cu at (139.7, 134.7)
- added R14: DNP, Resistor_SMD:R_0805_2012Metric, F.Cu at (137.3, 134.7)
- added R15: 120, Resistor_SMD:R_1206_3216Metric, F.Cu at (175.0, 140.7)
- added R16: 120, Resistor_SMD:R_1206_3216Metric, F.Cu at (81.6, 140.6)
- added U13: TJA1051T-3, Package_SO:SOIC-8_3.9x4.9mm_P1.27mm, F.Cu at (180.3, 140.6)
- added U14: WBO-Single-Module, wideband_module:f042_wideband_module, F.Cu at (60.3, 135.0)
- added U15: TJA1051T-3, Package_SO:SOIC-8_3.9x4.9mm_P1.27mm, F.Cu at (75.5, 140.3)
- moved R12 1.20 mm to (122.2, 51.8)
Connections:
- C1 pad 2: /12V_MR -> /12V_MR_FUSE
- C7 pad 2: /12V_MR -> /12V_MR_FUSE
- J4 pad 100: (no net) -> unconnected-(J4-Pad100)
- J4 pad 101: (no net) -> unconnected-(J4-Pad101)
- J4 pad 102: (no net) -> unconnected-(J4-Pad102)
- J4 pad 103: (no net) -> unconnected-(J4-Pad103)
- J4 pad 104: (no net) -> unconnected-(J4-Pad104)
- J4 pad 105: (no net) -> unconnected-(J4-Pad105)
- J4 pad 106: (no net) -> unconnected-(J4-Pad106)
- J4 pad 107: (no net) -> unconnected-(J4-Pad107)
- J4 pad 38: /5V_SENSOR_2 -> unconnected-(J4-Pad38)
- J4 pad 39: /5V_SENSOR_1 -> unconnected-(J4-Pad39)
- J4 pad 75: unconnected-(J4-Pad75) -> /RC1
- J4 pad 76: unconnected-(J4-Pad76) -> /RC2
- J4 pad 97: (no net) -> unconnected-(J4-Pad97)
- J4 pad 98: (no net) -> unconnected-(J4-Pad98)
- J4 pad 99: (no net) -> unconnected-(J4-Pad99)
- Motronic_88pin1 pad 10: /12V_MR -> /12V_MR_FUSE
- Motronic_88pin1 pad 37: /12V_MR -> /12V_MR_FUSE
- Motronic_88pin1 pad 68: /12V_MR -> /12V_MR_FUSE
- U1 pad 5: /CAN2+ -> /CAN_RX
- U1 pad 6: /CAN2- -> /CAN_TX
- U2 pad 4: /12V_MR -> /12V_MR_FUSE
- U8 pad 4: /12V_MR -> /12V_MR_FUSE
Routing:
- net /12V_MR_FUSE: track 100.9 -> 461.9 mm, vias 0 -> 8
- net /+3V3: track 123.1 -> 264.4 mm, vias 2 -> 4
- net /12V_MR: track 155.4 -> 21.0 mm, vias 3 -> 0
- net /+5V: track 58.5 -> 173.9 mm, vias 1 -> 2
- net /5V_SENSOR_2: track 280.6 -> 190.8 mm
- net /5V_SENSOR_1: track 180.9 -> 93.4 mm
- net /CAN2+: track 61.2 -> 123.4 mm, vias 0 -> 3
- net /CAN2-: track 66.8 -> 123.7 mm, vias 0 -> 3
- net GND: track 14.2 -> 61.8 mm, vias 496 -> 726
- net /CAN_TX: track 0.00 -> 21.7 mm
- net /CAN_RX: track 0.00 -> 20.1 mm
- net /IGN12: track 223.0 -> 207.1 mm
- net /IGN11: track 226.2 -> 211.4 mm
- net /IGN10: track 229.5 -> 216.3 mm
- net /IGN9: track 228.7 -> 217.4 mm
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