File: IGBT outputs.kicad_sch (KiCad schematic)
At the start: 16 parts, among them Q1 NGD8201AN, Q2 NGD8201AN, Q3 NGD8201AN, Q4 NGD8201AN, Q5 NGD8201AN, Q6 NGD8201AN, Q7 NGD8201AN, Q8 NGD8201AN

Commit message: schematic title blocks
Other:
- company: (none) -> FutureProofPerformance.com
- title: (none) -> Polygonus Universal 88p
Changed lines of the file:
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@@
 (kicad_sch (version 20230121) (generator eeschema)
   (paper "A4")
+  (title_block
+    (title "Polygonus Universal 88p")
+    (date "2023-11-12")
+    (rev "v1.0")
+    (company "FutureProofPerformance.com")
+  )
   (junction (at 215.9 71.12) (diameter 0) (color 0 0 0 0)
   )
