File: etb-9201.kicad_sch (KiCad schematic)
At the start: 5 parts, among them U2 TLE9201SG

Commit message: Competed board
Parts:
- renumbered C1 to C7, C2 to C8, C3 to C9, R1 to R12, U2 to U8
Changed lines of the file:
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@@
   (symbol (lib_id "Device:R") (at 68.58 57.15 270)
     (in_bom yes) (on_board yes)
-    (property "Reference" "R1" (id 0) (at 68.58 59.69 90))
+    (property "Reference" "R12" (id 0) (at 68.58 59.69 90))
     (property "Value" "10k" (id 1) (at 68.58 57.15 90))
     (property "Footprint" "Resistor_SMD:R_0402_1005Metric" (id 2) (at 68.58 55.372 90)
@@
   (symbol (lib_id "Simon:TLE9201SG") (at 97.79 63.5 0)
     (in_bom yes) (on_board yes) (fields_autoplaced)
-    (property "Reference" "U2" (id 0) (at 97.155 46.99 0))
+    (property "Reference" "U8" (id 0) (at 97.155 46.99 0))
     (property "Value" "TLE9201SG" (id 1) (at 97.155 49.53 0))
     (property "Footprint" "Package_SO:Infineon_PG-DSO-12-9" (id 2) (at 93.98 62.23 0)
@@
   (symbol (lib_id "Device:C_Small") (at 114.3 60.325 0)
     (in_bom yes) (on_board yes)
-    (property "Reference" "C3" (id 0) (at 116.6368 59.1566 0)
+    (property "Reference" "C9" (id 0) (at 116.6368 59.1566 0)
       (effects (font (size 1.27 1.27)) (justify left))
     )
@@
   (symbol (lib_id "Device:C") (at 80.645 46.99 0)
     (in_bom yes) (on_board yes)
-    (property "Reference" "C1" (id 0) (at 83.566 45.8216 0)
+    (property "Reference" "C7" (id 0) (at 83.566 45.8216 0)
       (effects (font (size 1.27 1.27)) (justify left))
     )
@@
   (symbol (lib_id "Device:C_Small") (at 114.3 48.895 0)
     (in_bom yes) (on_board yes)
-    (property "Reference" "C2" (id 0) (at 116.6368 47.7266 0)
+    (property "Reference" "C8" (id 0) (at 116.6368 47.7266 0)
       (effects (font (size 1.27 1.27)) (justify left))
     )

Commit message: updated and fixed, check JLC exports
Parts:
- C2: renamed from C8; footprint Capacitor_SMD:C_0603_1608Metric -> Capacitor_SMD:C_0805_2012Metric
- C3: renamed from C9; footprint Capacitor_SMD:C_0603_1608Metric -> Capacitor_SMD:C_0805_2012Metric
- R1: renamed from R12; footprint Resistor_SMD:R_0402_1005Metric -> Resistor_SMD:R_0805_2012Metric
- renumbered C7 to C1, U8 to U2
Changed lines of the file:
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@@
   (symbol (lib_id "Device:R") (at 68.58 57.15 270)
     (in_bom yes) (on_board yes)
-    (property "Reference" "R12" (id 0) (at 68.58 59.69 90))
+    (property "Reference" "R1" (id 0) (at 68.58 59.69 90))
     (property "Value" "10k" (id 1) (at 68.58 57.15 90))
-    (property "Footprint" "Resistor_SMD:R_0402_1005Metric" (id 2) (at 68.58 55.372 90)
+    (property "Footprint" "Resistor_SMD:R_0805_2012Metric" (id 2) (at 68.58 55.372 90)
       (effects (font (size 1.27 1.27)) hide)
     )
@@
   (symbol (lib_id "Simon:TLE9201SG") (at 97.79 63.5 0)
     (in_bom yes) (on_board yes) (fields_autoplaced)
-    (property "Reference" "U8" (id 0) (at 97.155 46.99 0))
+    (property "Reference" "U2" (id 0) (at 97.155 46.99 0))
     (property "Value" "TLE9201SG" (id 1) (at 97.155 49.53 0))
     (property "Footprint" "Package_SO:Infineon_PG-DSO-12-9" (id 2) (at 93.98 62.23 0)
@@
   (symbol (lib_id "Device:C_Small") (at 114.3 60.325 0)
     (in_bom yes) (on_board yes)
-    (property "Reference" "C9" (id 0) (at 116.6368 59.1566 0)
+    (property "Reference" "C3" (id 0) (at 116.6368 59.1566 0)
       (effects (font (size 1.27 1.27)) (justify left))
     )
@@
       (effects (font (size 1.27 1.27)) (justify left))
     )
-    (property "Footprint" "Capacitor_SMD:C_0603_1608Metric" (id 2) (at 114.3 60.325 0)
+    (property "Footprint" "Capacitor_SMD:C_0805_2012Metric" (id 2) (at 114.3 60.325 0)
       (effects (font (size 1.27 1.27)) hide)
     )
@@
   (symbol (lib_id "Device:C") (at 80.645 46.99 0)
     (in_bom yes) (on_board yes)
-    (property "Reference" "C7" (id 0) (at 83.566 45.8216 0)
+    (property "Reference" "C1" (id 0) (at 83.566 45.8216 0)
       (effects (font (size 1.27 1.27)) (justify left))
     )
@@
   (symbol (lib_id "Device:C_Small") (at 114.3 48.895 0)
     (in_bom yes) (on_board yes)
-    (property "Reference" "C8" (id 0) (at 116.6368 47.7266 0)
+    (property "Reference" "C2" (id 0) (at 116.6368 47.7266 0)
       (effects (font (size 1.27 1.27)) (justify left))
     )
@@
       (effects (font (size 1.27 1.27)) (justify left))
     )
-    (property "Footprint" "Capacitor_SMD:C_0603_1608Metric" (id 2) (at 114.3 48.895 0)
+    (property "Footprint" "Capacitor_SMD:C_0805_2012Metric" (id 2) (at 114.3 48.895 0)
       (effects (font (size 1.27 1.27)) hide)
     )

Commit message: All fixed up for JLC
Parts:
- C2, C3: LCSC C57112 -> C1710
- R1: LCSC C25744 -> C17414
Changed lines of the file:
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@@
       (effects (font (size 1.27 1.27)) hide)
     )
-    (property "LCSC" "C25744" (id 4) (at 68.58 57.15 0)
+    (property "LCSC" "C17414" (id 4) (at 68.58 57.15 0)
       (effects (font (size 1.27 1.27)) hide)
     )
@@
   (symbol (lib_id "power:GND") (at 85.09 74.93 270)
     (in_bom yes) (on_board yes)
-    (property "Reference" "#PWR051" (id 0) (at 78.74 74.93 0)
+    (property "Reference" "#PWR029" (id 0) (at 78.74 74.93 0)
       (effects (font (size 1.27 1.27)) hide)
     )
@@
   (symbol (lib_id "power:GND") (at 85.09 72.39 270)
     (in_bom yes) (on_board yes)
-    (property "Reference" "#PWR050" (id 0) (at 78.74 72.39 0)
+    (property "Reference" "#PWR028" (id 0) (at 78.74 72.39 0)
       (effects (font (size 1.27 1.27)) hide)
     )
@@
   (symbol (lib_id "power:GND") (at 114.3 62.865 0)
     (in_bom yes) (on_board yes)
-    (property "Reference" "#PWR053" (id 0) (at 114.3 69.215 0)
+    (property "Reference" "#PWR031" (id 0) (at 114.3 69.215 0)
       (effects (font (size 1.27 1.27)) hide)
     )
@@
   (symbol (lib_id "power:GND") (at 114.3 46.355 180)
     (in_bom yes) (on_board yes)
-    (property "Reference" "#PWR052" (id 0) (at 114.3 40.005 0)
+    (property "Reference" "#PWR030" (id 0) (at 114.3 40.005 0)
       (effects (font (size 1.27 1.27)) hide)
     )
@@
       (effects (font (size 1.27 1.27)) hide)
     )
-    (property "LCSC" "C57112" (id 5) (at 114.3 60.325 0)
+    (property "LCSC" "C1710" (id 5) (at 114.3 60.325 0)
       (effects (font (size 1.27 1.27)) hide)
     )
@@
       (effects (font (size 1.27 1.27)) hide)
     )
-    (property "LCSC" "C57112" (id 5) (at 114.3 48.895 0)
+    (property "LCSC" "C1710" (id 5) (at 114.3 48.895 0)
       (effects (font (size 1.27 1.27)) hide)
     )
@@
   (symbol (lib_id "power:GND") (at 80.645 43.18 180)
     (in_bom yes) (on_board yes)
-    (property "Reference" "#PWR049" (id 0) (at 80.645 36.83 0)
+    (property "Reference" "#PWR027" (id 0) (at 80.645 36.83 0)
       (effects (font (size 1.27 1.27)) hide)
     )

Commit message: Fixed 12V_RAW and added grounds for sensors
Parts:
- renumbered C1 to C7, C2 to C8, C3 to C9, R1 to R12, U2 to U8
Changed lines of the file:
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@@
   (symbol (lib_id "Device:R") (at 68.58 57.15 270)
     (in_bom yes) (on_board yes)
-    (property "Reference" "R1" (id 0) (at 68.58 59.69 90))
+    (property "Reference" "R12" (id 0) (at 68.58 59.69 90))
     (property "Value" "10k" (id 1) (at 68.58 57.15 90))
     (property "Footprint" "Resistor_SMD:R_0805_2012Metric" (id 2) (at 68.58 55.372 90)
@@
   (symbol (lib_id "power:GND") (at 85.09 74.93 270)
     (in_bom yes) (on_board yes)
-    (property "Reference" "#PWR029" (id 0) (at 78.74 74.93 0)
+    (property "Reference" "#PWR051" (id 0) (at 78.74 74.93 0)
       (effects (font (size 1.27 1.27)) hide)
     )
@@
   (symbol (lib_id "power:GND") (at 85.09 72.39 270)
     (in_bom yes) (on_board yes)
-    (property "Reference" "#PWR028" (id 0) (at 78.74 72.39 0)
+    (property "Reference" "#PWR050" (id 0) (at 78.74 72.39 0)
       (effects (font (size 1.27 1.27)) hide)
     )
@@
   (symbol (lib_id "power:GND") (at 114.3 62.865 0)
     (in_bom yes) (on_board yes)
-    (property "Reference" "#PWR031" (id 0) (at 114.3 69.215 0)
+    (property "Reference" "#PWR053" (id 0) (at 114.3 69.215 0)
       (effects (font (size 1.27 1.27)) hide)
     )
@@
   (symbol (lib_id "power:GND") (at 114.3 46.355 180)
     (in_bom yes) (on_board yes)
-    (property "Reference" "#PWR030" (id 0) (at 114.3 40.005 0)
+    (property "Reference" "#PWR052" (id 0) (at 114.3 40.005 0)
       (effects (font (size 1.27 1.27)) hide)
     )
@@
   (symbol (lib_id "Simon:TLE9201SG") (at 97.79 63.5 0)
     (in_bom yes) (on_board yes) (fields_autoplaced)
-    (property "Reference" "U2" (id 0) (at 97.155 46.99 0))
+    (property "Reference" "U8" (id 0) (at 97.155 46.99 0))
     (property "Value" "TLE9201SG" (id 1) (at 97.155 49.53 0))
     (property "Footprint" "Package_SO:Infineon_PG-DSO-12-9" (id 2) (at 93.98 62.23 0)
@@
   (symbol (lib_id "Device:C_Small") (at 114.3 60.325 0)
     (in_bom yes) (on_board yes)
-    (property "Reference" "C3" (id 0) (at 116.6368 59.1566 0)
+    (property "Reference" "C9" (id 0) (at 116.6368 59.1566 0)
       (effects (font (size 1.27 1.27)) (justify left))
     )
@@
   (symbol (lib_id "Device:C") (at 80.645 46.99 0)
     (in_bom yes) (on_board yes)
-    (property "Reference" "C1" (id 0) (at 83.566 45.8216 0)
+    (property "Reference" "C7" (id 0) (at 83.566 45.8216 0)
       (effects (font (size 1.27 1.27)) (justify left))
     )
@@
   (symbol (lib_id "Device:C_Small") (at 114.3 48.895 0)
     (in_bom yes) (on_board yes)
-    (property "Reference" "C2" (id 0) (at 116.6368 47.7266 0)
+    (property "Reference" "C8" (id 0) (at 116.6368 47.7266 0)
       (effects (font (size 1.27 1.27)) (justify left))
     )
@@
   (symbol (lib_id "power:GND") (at 80.645 43.18 180)
     (in_bom yes) (on_board yes)
-    (property "Reference" "#PWR027" (id 0) (at 80.645 36.83 0)
+    (property "Reference" "#PWR049" (id 0) (at 80.645 36.83 0)
       (effects (font (size 1.27 1.27)) hide)
     )

Commit message: convert to kicad7, add jumpers for direct drive igbt output
Parts:
- renumbered C7 to C1, C8 to C2, C9 to C3, R12 to R1, U8 to U2

Commit message: fix wideband library, ERC, DRC
Connections:
- net 3.3V renamed +3.3V

Commit message: schematic title blocks
Other:
- company: (none) -> FutureProofPerformance.com
- title: (none) -> Polygonus Universal 88p
Changed lines of the file:
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@@
 (kicad_sch (version 20230121) (generator eeschema)
   (paper "A4")
+  (title_block
+    (title "Polygonus Universal 88p")
+    (date "2023-11-12")
+    (rev "v1.0")
+    (company "FutureProofPerformance.com")
+  )
   (junction (at 80.645 53.34) (diameter 0) (color 0 0 0 0)
   )
