File: Polygonus-Universal-Base.kicad_sch (KiCad schematic)
At the start: 14 parts, among them J4 Polygonus_Plugs, U1 f042_wideband_module, U14 f042_wideband_module

Commit message: fixed stepper pullup and updated silkscreen
Parts:
- added R17, R18: 1k, Resistor_SMD:R_0805_2012Metric, symbol hellen-one-common:Res
Connections:
- net +5V: now also R17.1, R18.2
- net LS10: now also R17.2
- net LS9: now also R18.1
Changed lines of the file:
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@@
+    (stroke (width 0) (type default))
+  )
+  (wire (pts (xy 33.02 240.03) (xy 33.02 242.57))
     (stroke (width 0) (type default))
   )
@@
     (stroke (width 0) (type default))
   )
+  (wire (pts (xy 33.02 240.03) (xy 38.1 240.03))
+    (stroke (width 0) (type default))
+  )
   (wire (pts (xy 271.78 45.72) (xy 279.4 45.72))
     (stroke (width 0) (type default))
@@
     (stroke (width 0) (type default))
   )
+  (wire (pts (xy 33.02 233.68) (xy 33.02 237.49))
+    (stroke (width 0) (type default))
+  )
   (wire (pts (xy 279.4 262.89) (xy 271.78 262.89))
     (stroke (width 0) (type default))
@@
   )
   (wire (pts (xy 271.78 35.56) (xy 279.4 35.56))
+    (stroke (width 0) (type default))
+  )
+  (wire (pts (xy 33.02 237.49) (xy 38.1 237.49))
     (stroke (width 0) (type default))
   )
@@
     (effects (font (size 1.27 1.27)) (justify right bottom))
   )
+  (label "+5V" (at 22.86 233.68 180) (fields_autoplaced)
+    (effects (font (size 1.27 1.27)) (justify right bottom))
+  )
   (label "IGN12" (at 130.81 113.03 180) (fields_autoplaced)
     (effects (font (size 1.27 1.27)) (justify right bottom))
@@
   )
   (label "LSU_Un" (at 271.78 76.2 180) (fields_autoplaced)
+    (effects (font (size 1.27 1.27)) (justify right bottom))
+  )
+  (label "+5V" (at 22.86 242.57 180) (fields_autoplaced)
     (effects (font (size 1.27 1.27)) (justify right bottom))
   )
@@
     )
   )
+  (symbol (lib_id "hellen-one-common:Res") (at 33.02 233.68 0) (mirror y) (unit 1)
+    (in_bom yes) (on_board yes) (dnp no)
+    (property "Reference" "R18" (at 27.94 231.14 0)
+      (effects (font (size 1.27 1.27)))
+    )
+    (property "Value" "1k" (at 27.94 233.68 0)
+      (effects (font (size 1.27 1.27)))
+    )
+    (property "Footprint" "Resistor_SMD:R_0805_2012Metric" (at 29.21 237.49 0)
+      (effects (font (size 1.27 1.27)) hide)
+    )
+    (property "Datasheet" "" (at 33.02 233.68 0)
+      (effects (font (size 1.27 1.27)) hide)
+    )
+    (property "LCSC" "C21190" (at 33.02 233.68 0)
+      (effects (font (size 1.27 1.27)) hide)
+    )
+    (pin "1")
+    (pin "2")
+    (instances
+      (project "Polygonus-Universal-Base"
+        (path "/e63e39d7-6ac0-4ffd-8aa3-1841a4541b55"
+          (reference "R18") (unit 1)
+        )
+      )
+    )
+  )
   (symbol (lib_name "GND_1") (lib_id "power:GND") (at 271.78 151.13 270) (unit 1)
     (in_bom yes) (on_board yes) (dnp no) (fields_autoplaced)
@@
         )
       )
+    )
+  )
+  (symbol (lib_id "hellen-one-common:Res") (at 22.86 242.57 0) (mirror x) (unit 1)
+    (in_bom yes) (on_board yes) (dnp no)
+    (property "Reference" "R17" (at 27.94 245.11 0)
+      (effects (font (size 1.27 1.27)))
+    )
+    (property "Value" "1k" (at 27.94 242.57 0)
+      (effects (font (size 1.27 1.27)))
+    )
+    (property "Footprint" "Resistor_SMD:R_0805_2012Metric" (at 26.67 238.76 0)
+      (effects (font (size 1.27 1.27)) hide)
+    )
+    (property "Datasheet" "" (at 22.86 242.57 0)
+      (effects (font (size 1.27 1.27)) hide)
+    )
+    (property "LCSC" "C21190" (at 22.86 242.57 0)
+      (effects (font (size 1.27 1.27)) hide)
+    )
+    (pin "1")
+    (pin "2")
+    (instances
+      (project "Polygonus-Universal-Base"
+        (path "/e63e39d7-6ac0-4ffd-8aa3-1841a4541b55"
+          (reference "R17") (unit 1)
+        )
+      )
